Commit message: Fixing package's names.

File: src/depth_image_forecasting/urdf/ABot.urdf.xacro (robot description, xacro)
@@ -236,5 +236,5 @@
       <origin xyz="0 0 0" rpy="0 0 0"/>
       <geometry>
-        <mesh filename="package://gazebo_demo/urdf/hokuyo.dae"/>
+        <mesh filename="package://depth_image_forecasting/urdf/hokuyo.dae"/>
       </geometry>
     </visual>
